File: hw/uDC_module.brd (EAGLE design)
At the start: 25 x 45 mm, 38 parts, among them J1 GROVE-4P-2.0-3470130P1, J2 GROVE-4P-2.0-3470130P1, U5 LD3985XX, X1 22-23-2021, X2 22-23-2021, X3 53047-06, X4 53047-06

Commit message: final revision
Connections:
- net +5V: now also X4.1; no longer X4.2
- net GND: now also X3.2, X3.4, X3.6, X4.2; no longer X3.1, X3.3, X3.5, X4.1
- net LIMIT_A: now also X3.1; no longer X3.2
- net LIMIT_B: now also X3.3; no longer X3.4
- net STOP: now also X3.5; no longer X3.6
Routing:
- net +5V: track 71.1 -> 72.3 mm
- net LIMIT_B: track 26.4 -> 25.9 mm
- net STOP: track 26.5 -> 26.0 mm
- net LIMIT_A: track 24.4 -> 25.0 mm
Changed lines of the file:
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@@
 <grid distance="0.5" unitdist="mm" unit="mm" style="dots" multiple="1" display="yes" altdistance="0.1" altunitdist="mm" altunit="mm"/>
 <layers>
-<layer number="1" name="Top" color="4" fill="1" visible="no" active="yes"/>
-<layer number="16" name="Bottom" color="1" fill="1" visible="yes" active="yes"/>
+<layer number="1" name="Top" color="4" fill="1" visible="yes" active="yes"/>
+<layer number="16" name="Bottom" color="1" fill="1" visible="no" active="yes"/>
 <layer number="17" name="Pads" color="2" fill="1" visible="yes" active="yes"/>
 <layer number="18" name="Vias" color="2" fill="1" visible="yes" active="yes"/>
 <layer number="19" name="Unrouted" color="6" fill="1" visible="yes" active="yes"/>
 <layer number="20" name="Dimension" color="15" fill="1" visible="yes" active="yes"/>
-<layer number="21" name="tPlace" color="7" fill="1" visible="no" active="yes"/>
-<layer number="22" name="bPlace" color="7" fill="1" visible="yes" active="yes"/>
-<layer number="23" name="tOrigins" color="15" fill="1" visible="no" active="yes"/>
-<layer number="24" name="bOrigins" color="15" fill="1" visible="yes" active="yes"/>
+<layer number="21" name="tPlace" color="7" fill="1" visible="yes" active="yes"/>
+<layer number="22" name="bPlace" color="7" fill="1" visible="no" active="yes"/>
+<layer number="23" name="tOrigins" color="15" fill="1" visible="yes" active="yes"/>
+<layer number="24" name="bOrigins" color="15" fill="1" visible="no" active="yes"/>
 <layer number="25" name="tNames" color="7" fill="1" visible="no" active="yes"/>
 <layer number="26" name="bNames" color="7" fill="1" visible="no" active="yes"/>
@@
 <layer number="37" name="tTest" color="7" fill="1" visible="no" active="yes"/>
 <layer number="38" name="bTest" color="7" fill="1" visible="no" active="yes"/>
-<layer number="39" name="tKeepout" color="4" fill="11" visible="no" active="yes"/>
-<layer number="40" name="bKeepout" color="1" fill="11" visible="yes" active="yes"/>
-<layer number="41" name="tRestrict" color="4" fill="10" visible="no" active="yes"/>
-<layer number="42" name="bRestrict" color="1" fill="10" visible="yes" active="yes"/>
+<layer number="39" name="tKeepout" color="4" fill="11" visible="yes" active="yes"/>
+<layer number="40" name="bKeepout" color="1" fill="11" visible="no" active="yes"/>
+<layer number="41" name="tRestrict" color="4" fill="10" visible="yes" active="yes"/>
+<layer number="42" name="bRestrict" color="1" fill="10" visible="no" active="yes"/>
 <layer number="43" name="vRestrict" color="2" fill="10" visible="no" active="yes"/>
 <layer number="44" name="Drills" color="7" fill="1" visible="no" active="yes"/>
@@
 <layer number="46" name="Milling" color="3" fill="1" visible="yes" active="yes"/>
 <layer number="47" name="Measures" color="7" fill="1" visible="no" active="yes"/>
-<layer number="48" name="Document" color="7" fill="1" visible="no" active="yes"/>
+<layer number="48" name="Document" color="7" fill="1" visible="yes" active="yes"/>
 <layer number="49" name="Reference" color="7" fill="1" visible="no" active="yes"/>
 <layer number="50" name="dxf" color="7" fill="1" visible="no" active="no"/>
-<layer number="51" name="tDocu" color="7" fill="1" visible="no" active="yes"/>
-<layer number="52" name="bDocu" color="7" fill="1" visible="yes" active="yes"/>
+<layer number="51" name="tDocu" color="7" fill="1" visible="yes" active="yes"/>
+<layer number="52" name="bDocu" color="7" fill="1" visible="no" active="yes"/>
 <layer number="53" name="tGND_GNDA" color="7" fill="1" visible="no" active="no"/>
 <layer number="54" name="bGND_GNDA" color="7" fill="1" visible="no" active="no"/>
@@
 <via x="17.3" y="22.9" extent="1-16" drill="0.3"/>
 <via x="18.1" y="11.2" extent="1-16" drill="0.3"/>
-<contactref element="X4" pad="1"/>
-<contactref element="X3" pad="1"/>
-<contactref element="X3" pad="3"/>
-<contactref element="X3" pad="5"/>
+<contactref element="X4" pad="2"/>
+<contactref element="X3" pad="2"/>
+<contactref element="X3" pad="4"/>
+<contactref element="X3" pad="6"/>
 </signal>
 <signal name="VIN">
@@
 <wire x1="0.7" y1="39.4" x2="0.7" y2="43" width="0.4" layer="1"/>
 <wire x1="0.7" y1="43" x2="2" y2="44.3" width="0.4" layer="1"/>
-<contactref element="X4" pad="2"/>
-<wire x1="20.375" y1="42.85" x2="20.375" y2="43.625" width="0.4" layer="1"/>
-<wire x1="20.375" y1="43.625" x2="19.7" y2="44.3" width="0.4" layer="1"/>
-<wire x1="19.7" y1="44.3" x2="2" y2="44.3" width="0.4" layer="1"/>
+<wire x1="20.9" y1="44.3" x2="2" y2="44.3" width="0.4" layer="1"/>
+<contactref element="X4" pad="1"/>
+<wire x1="21.625" y1="42.85" x2="21.625" y2="43.575" width="0.4" layer="1"/>
+<wire x1="21.625" y1="43.575" x2="20.9" y2="44.3" width="0.4" layer="1"/>
 </signal>
 <signal name="D1">
@@
 <wire x1="16.3" y1="19.8" x2="17.2" y2="20.7" width="0.2" layer="16"/>
 <wire x1="17.2" y1="20.7" x2="17.9" y2="20.7" width="0.2" layer="16"/>
-<contactref element="X3" pad="6"/>
-<wire x1="19.4" y1="32.5" x2="19.4" y2="34.6" width="0.2" layer="16"/>
-<wire x1="15.375" y1="39.45" x2="15.375" y2="38.625" width="0.2" layer="16"/>
-<wire x1="15.375" y1="38.625" x2="19.4" y2="34.6" width="0.2" layer="16"/>
+<contactref element="X3" pad="5"/>
+<wire x1="19.4" y1="32.5" x2="19.4" y2="35.8" width="0.2" layer="16"/>
+<wire x1="19.4" y1="35.8" x2="16.7" y2="38.5" width="0.2" layer="16"/>
+<wire x1="16.625" y1="39.45" x2="16.625" y2="38.575" width="0.2" layer="16"/>
+<wire x1="16.625" y1="38.575" x2="16.7" y2="38.5" width="0.2" layer="16"/>
 </signal>
 <signal name="LIMIT_B">
@@
 <wire x1="18.1" y1="20.3" x2="22.5" y2="24.7" width="0.2" layer="16"/>
 <wire x1="22.5" y1="24.7" x2="22.5" y2="30" width="0.2" layer="16"/>
-<contactref element="X3" pad="4"/>
-<wire x1="19.8" y1="32.7" x2="19.8" y2="36.7" width="0.2" layer="16"/>
-<wire x1="17.875" y1="39.45" x2="17.875" y2="38.625" width="0.2" layer="16"/>
-<wire x1="17.875" y1="38.625" x2="19.8" y2="36.7" width="0.2" layer="16"/>
+<contactref element="X3" pad="3"/>
+<wire x1="19.8" y1="32.7" x2="19.8" y2="37.9" width="0.2" layer="16"/>
+<wire x1="19.8" y1="37.9" x2="19.2" y2="38.5" width="0.2" layer="16"/>
+<wire x1="19.125" y1="39.45" x2="19.125" y2="38.575" width="0.2" layer="16"/>
+<wire x1="19.125" y1="38.575" x2="19.2" y2="38.5" width="0.2" layer="16"/>
 </signal>
 <signal name="LIMIT_A">
@@
 <wire x1="18.1" y1="19.7" x2="22.9" y2="24.5" width="0.2" layer="16"/>
 <wire x1="22.9" y1="24.5" x2="22.9" y2="30.2" width="0.2" layer="16"/>
-<contactref element="X3" pad="2"/>
-<wire x1="20.2" y1="32.9" x2="20.2" y2="38.4" width="0.2" layer="16"/>
-<wire x1="20.375" y1="39.45" x2="20.375" y2="38.575" width="0.2" layer="16"/>
-<wire x1="20.375" y1="38.575" x2="20.2" y2="38.4" width="0.2" layer="16"/>
+<contactref element="X3" pad="1"/>
+<wire x1="20.2" y1="32.9" x2="20.2" y2="37.1" width="0.2" layer="16"/>
+<wire x1="20.2" y1="37.1" x2="21.6" y2="38.5" width="0.2" layer="16"/>
+<wire x1="21.625" y1="39.45" x2="21.625" y2="38.525" width="0.2" layer="16"/>
+<wire x1="21.625" y1="38.525" x2="21.6" y2="38.5" width="0.2" layer="16"/>
 </signal>
 </signals>
