File: hw/uDC_module.sch (EAGLE design)
At the start: 23 parts, among them J1 GROVE-4P-2.0-3470130P1, J2 GROVE-4P-2.0-3470130P1

Commit message: ongoing layout
Parts:
- added C10, C11: (no value), rcl:CPOL-EUD
- added C12: 33n, rcl:C-EUC0603
- added C13, C15: 100n, rcl:C-EUC0603
- added R2: 10k, rcl:R-EU_R0603
- added U$7: MC33962, freescale:MC33962
- added X1, X2: 22-23-2021, con-molex:22-23-2021
- added X3, X4: 53047-06, con-molex:53047-06
Connections:
- new net +V: C10.+, C11.+, C12.1, C13.1, U$7.VPWR, X1-1.S
- new net MA: U$7.OUT1, X2-1.S
- new net MB: U$7.OUT2, X2-2.S
- new net N$10: U$7.INV
- new net N$11: U$7.D1
- new net N$12: U$7.!D2
- new net N$13: U$7.IN2
- new net N$14: U$7.IN1
- new net N$15: U$7.EN
- new net N$3: C15.1, R2.2, U$7.FB
- new net N$5: U$7.!SF
- new net N$6: C12.2, U$7.CCP
- new net N$9: U$7.SLEW
- net GND: now also C10.-, C11.-, C13.2, C15.2, R2.1, U$7.AGND, U$7.PGND, X1-2.S
Changed lines of the file:
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@@
 <part name="U$1" library="r2p_pcb" deviceset="PCB_25X45" device=""/>
 <part name="U$5" library="abracon" deviceset="ASD" device=""/>
+<part name="C10" library="rcl" deviceset="CPOL-EU" device="D"/>
+<part name="C11" library="rcl" deviceset="CPOL-EU" device="D"/>
+<part name="GND15" library="supply" deviceset="GND" device=""/>
+<part name="X1" library="con-molex" deviceset="22-23-2021" device=""/>
+<part name="X2" library="con-molex" deviceset="22-23-2021" device=""/>
+<part name="X3" library="con-molex" deviceset="53?-06" device="047"/>
+<part name="C12" library="rcl" deviceset="C-EU" device="C0603" value="33n"/>
+<part name="GND18" library="supply1" deviceset="GND" device=""/>
+<part name="P+1" library="supply" deviceset="+V" device=""/>
+<part name="P+2" library="supply" deviceset="+V" device=""/>
+<part name="GND20" library="supply" deviceset="GND" device=""/>
+<part name="U$7" library="freescale" deviceset="MC33962" device=""/>
+<part name="C13" library="rcl" deviceset="C-EU" device="C0603" value="100n"/>
+<part name="GND21" library="supply1" deviceset="GND" device=""/>
+<part name="C15" library="rcl" deviceset="C-EU" device="C0603" value="100n"/>
+<part name="R2" library="rcl" deviceset="R-EU_" device="R0603" value="10k"/>
+<part name="GND23" library="supply" deviceset="GND" device=""/>
+<part name="GND24" library="supply" deviceset="GND" device=""/>
+<part name="X4" library="con-molex" deviceset="53?-06" device="047"/>
+<part name="GND14" library="supply" deviceset="GND" device=""/>
 </parts>
 <sheets>
@@
 <instance part="U$1" gate="A" x="27.94" y="22.86"/>
 <instance part="U$5" gate="G$1" x="116.84" y="170.18"/>
+<instance part="C10" gate="G$1" x="304.8" y="144.78"/>
+<instance part="C11" gate="G$1" x="294.64" y="144.78"/>
+<instance part="GND15" gate="1" x="243.84" y="170.18"/>
+<instance part="X1" gate="-1" x="317.5" y="144.78"/>
+<instance part="X1" gate="-2" x="317.5" y="142.24"/>
+<instance part="X2" gate="-1" x="317.5" y="127"/>
+<instance part="X2" gate="-2" x="317.5" y="124.46"/>
+<instance part="X3" gate="-1" x="271.78" y="124.46"/>
+<instance part="X3" gate="-2" x="271.78" y="121.92"/>
+<instance part="X3" gate="-3" x="271.78" y="119.38"/>
+<instance part="X3" gate="-4" x="271.78" y="116.84"/>
+<instance part="X3" gate="-5" x="271.78" y="114.3"/>
+<instance part="X3" gate="-6" x="271.78" y="111.76"/>
+<instance part="C12" gate="G$1" x="248.92" y="198.12"/>
+<instance part="GND18" gate="1" x="304.8" y="137.16"/>
+<instance part="P+1" gate="1" x="243.84" y="208.28"/>
+<instance part="P+2" gate="1" x="312.42" y="152.4"/>
+<instance part="GND20" gate="1" x="312.42" y="137.16"/>
+<instance part="U$7" gate="G$1" x="223.52" y="185.42"/>
+<instance part="C13" gate="G$1" x="284.48" y="144.78"/>
+<instance part="GND21" gate="1" x="284.48" y="137.16"/>
+<instance part="C15" gate="G$1" x="200.66" y="172.72"/>
+<instance part="R2" gate="G$1" x="193.04" y="170.18" rot="R90"/>
+<instance part="GND23" gate="1" x="200.66" y="162.56"/>
+<instance part="GND24" gate="1" x="193.04" y="162.56"/>
+<instance part="X4" gate="-1" x="233.68" y="109.22"/>
+<instance part="X4" gate="-2" x="233.68" y="106.68"/>
+<instance part="X4" gate="-3" x="233.68" y="104.14"/>
+<instance part="X4" gate="-4" x="233.68" y="101.6"/>
+<instance part="X4" gate="-5" x="233.68" y="99.06"/>
+<instance part="X4" gate="-6" x="233.68" y="96.52"/>
+<instance part="GND14" gate="1" x="294.64" y="137.16"/>
 </instances>
 <busses>
@@
 <wire x1="76.2" y1="66.04" x2="76.2" y2="63.5" width="0.1524" layer="91"/>
 <pinref part="SOT1" gate="G$1" pin="RS"/>
+</segment>
+<segment>
+<pinref part="C10" gate="G$1" pin="-"/>
+<pinref part="GND18" gate="1" pin="GND"/>
+</segment>
+<segment>
+<pinref part="X1" gate="-2" pin="S"/>
+<pinref part="GND20" gate="1" pin="GND"/>
+<wire x1="314.96" y1="142.24" x2="312.42" y2="142.24" width="0.1524" layer="91"/>
+<wire x1="312.42" y1="142.24" x2="312.42" y2="139.7" width="0.1524" layer="91"/>
+</segment>
+<segment>
+<pinref part="C13" gate="G$1" pin="2"/>
+<pinref part="GND21" gate="1" pin="GND"/>
+</segment>
+<segment>
+<pinref part="C15" gate="G$1" pin="2"/>
+<pinref part="GND23" gate="1" pin="GND"/>
+<wire x1="200.66" y1="165.1" x2="200.66" y2="167.64" width="0.1524" layer="91"/>
+</segment>
+<segment>
+<pinref part="R2" gate="G$1" pin="1"/>
+<pinref part="GND24" gate="1" pin="GND"/>
+</segment>
+<segment>
+<pinref part="U$7" gate="G$1" pin="AGND"/>
+<pinref part="GND15" gate="1" pin="GND"/>
+<wire x1="241.3" y1="177.8" x2="243.84" y2="177.8" width="0.1524" layer="91"/>
+<wire x1="243.84" y1="177.8" x2="243.84" y2="175.26" width="0.1524" layer="91"/>
+<pinref part="U$7" gate="G$1" pin="PGND"/>
+<wire x1="243.84" y1="175.26" x2="243.84" y2="172.72" width="0.1524" layer="91"/>
+<wire x1="241.3" y1="175.26" x2="243.84" y2="175.26" width="0.1524" layer="91"/>
+<junction x="243.84" y="175.26"/>
+</segment>
+<segment>
+<pinref part="C11" gate="G$1" pin="-"/>
+<pinref part="GND14" gate="1" pin="GND"/>
 </segment>
 </net>
@@
 </segment>
 </net>
+<net name="N$6" class="0">
+<segment>
+<pinref part="C12" gate="G$1" pin="2"/>
+<wire x1="241.3" y1="193.04" x2="248.92" y2="193.04" width="0.1524" layer="91"/>
+<pinref part="U$7" gate="G$1" pin="CCP"/>
+</segment>
+</net>
+<net name="+V" class="0">
+<segment>
+<wire x1="241.3" y1="195.58" x2="243.84" y2="195.58" width="0.1524" layer="91"/>
+<wire x1="243.84" y1="195.58" x2="243.84" y2="200.66" width="0.1524" layer="91"/>
+<pinref part="C12" gate="G$1" pin="1"/>
+<wire x1="243.84" y1="200.66" x2="243.84" y2="205.74" width="0.1524" layer="91"/>
+<wire x1="248.92" y1="200.66" x2="243.84" y2="200.66" width="0.1524" layer="91"/>
+<junction x="243.84" y="200.66"/>
+<pinref part="P+1" gate="1" pin="+V"/>
+<pinref part="U$7" gate="G$1" pin="VPWR"/>
+</segment>
+<segment>
+<pinref part="P+2" gate="1" pin="+V"/>
+<pinref part="X1" gate="-1" pin="S"/>
+<wire x1="314.96" y1="144.78" x2="312.42" y2="144.78" width="0.1524" layer="91"/>
+<wire x1="312.42" y1="144.78" x2="312.42" y2="147.32" width="0.1524" layer="91"/>
+<pinref part="C13" gate="G$1" pin="1"/>
+<wire x1="312.42" y1="147.32" x2="312.42" y2="149.86" width="0.1524" layer="91"/>
+<wire x1="284.48" y1="147.32" x2="294.64" y2="147.32" width="0.1524" layer="91"/>
+<pinref part="C10" gate="G$1" pin="+"/>
+<wire x1="294.64" y1="147.32" x2="304.8" y2="147.32" width="0.1524" layer="91"/>
+<wire x1="304.8" y1="147.32" x2="312.42" y2="147.32" width="0.1524" layer="91"/>
+<junction x="304.8" y="147.32"/>
+<junction x="312.42" y="147.32"/>
+<pinref part="C11" gate="G$1" pin="+"/>
+<junction x="294.64" y="147.32"/>
+</segment>
+</net>
+<net name="MA" class="0">
+<segment>
+<wire x1="241.3" y1="185.42" x2="243.84" y2="185.42" width="0.1524" layer="91"/>
+<pinref part="U$7" gate="G$1" pin="OUT1"/>
+<label x="243.84" y="185.42" size="1.778" layer="95"/>
+</segment>
+<segment>
+<pinref part="X2" gate="-1" pin="S"/>
+<wire x1="314.96" y1="127" x2="309.88" y2="127" width="0.1524" layer="91"/>
+<label x="309.88" y="127" size="1.778" layer="95" rot="MR0"/>
+</segment>
+</net>
+<net name="MB" class="0">
+<segment>
+<wire x1="241.3" y1="182.88" x2="243.84" y2="182.88" width="0.1524" layer="91"/>
+<pinref part="U$7" gate="G$1" pin="OUT2"/>
+<label x="243.84" y="182.88" size="1.778" layer="95"/>
+</segment>
+<segment>
+<pinref part="X2" gate="-2" pin="S"/>
+<wire x1="314.96" y1="124.46" x2="309.88" y2="124.46" width="0.1524" layer="91"/>
+<label x="309.88" y="124.46" size="1.778" layer="95" rot="MR0"/>
+</segment>
+</net>
+<net name="N$3" class="0">
+<segment>
+<pinref part="U$7" gate="G$1" pin="FB"/>
+<wire x1="205.74" y1="175.26" x2="200.66" y2="175.26" width="0.1524" layer="91"/>
+<pinref part="C15" gate="G$1" pin="1"/>
+<wire x1="200.66" y1="175.26" x2="193.04" y2="175.26" width="0.1524" layer="91"/>
+<junction x="200.66" y="175.26"/>
+<pinref part="R2" gate="G$1" pin="2"/>
+<wire x1="193.04" y1="175.26" x2="187.96" y2="175.26" width="0.1524" layer="91"/>
+<junction x="193.04" y="175.26"/>
+<label x="187.96" y="175.26" size="1.778" layer="95" rot="MR0"/>
+</segment>
+</net>
+<net name="N$5" class="0">
+<segment>
+<pinref part="U$7" gate="G$1" pin="!SF"/>
+<wire x1="205.74" y1="177.8" x2="203.2" y2="177.8" width="0.1524" layer="91"/>
+</segment>
+</net>
+<net name="N$9" class="0">
+<segment>
+<pinref part="U$7" gate="G$1" pin="SLEW"/>
+<wire x1="205.74" y1="180.34" x2="203.2" y2="180.34" width="0.1524" layer="91"/>
+</segment>
+</net>
+<net name="N$10" class="0">
+<segment>
+<pinref part="U$7" gate="G$1" pin="INV"/>
+<wire x1="205.74" y1="182.88" x2="203.2" y2="182.88" width="0.1524" layer="91"/>
+</segment>
+</net>
+<net name="N$11" class="0">
+<segment>
+<pinref part="U$7" gate="G$1" pin="D1"/>
+<wire x1="205.74" y1="185.42" x2="203.2" y2="185.42" width="0.1524" layer="91"/>
+</segment>
+</net>
+<net name="N$12" class="0">
+<segment>
+<pinref part="U$7" gate="G$1" pin="!D2"/>
+<wire x1="205.74" y1="187.96" x2="203.2" y2="187.96" width="0.1524" layer="91"/>
+</segment>
+</net>
+<net name="N$13" class="0">
+<segment>
+<pinref part="U$7" gate="G$1" pin="IN2"/>
+<wire x1="205.74" y1="190.5" x2="203.2" y2="190.5" width="0.1524" layer="91"/>
+</segment>
+</net>
+<net name="N$14" class="0">
+<segment>
+<pinref part="U$7" gate="G$1" pin="IN1"/>
+<wire x1="205.74" y1="193.04" x2="203.2" y2="193.04" width="0.1524" layer="91"/>
+</segment>
+</net>
+<net name="N$15" class="0">
+<segment>
+<pinref part="U$7" gate="G$1" pin="EN"/>
+<wire x1="205.74" y1="195.58" x2="203.2" y2="195.58" width="0.1524" layer="91"/>
+</segment>
+</net>

Commit message: ongoing layout
Parts:
- U$6: value STM32F103CX -> STM32F103CXTX; device st:STM32F103CX -> st:STM32F103CXTX
Connections:
- net N$10 renamed INV
- net N$11 renamed D1
- net N$12 renamed !D2
- net N$13 renamed IN2
- net N$14 renamed IN1
- net N$15 renamed EN
- net N$3 renamed FB
- net N$5 renamed !SF
- net N$9 renamed SLEW
Changed lines of the file:
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@@
 <part name="J1" library="OPL Eagle Library" deviceset="GROVE-4P-2.0" device="-3470130P1"/>
 <part name="+3V7" library="supply1" deviceset="+3V3" device=""/>
-<part name="U$6" library="st" deviceset="STM32F103CX" device=""/>
+<part name="U$6" library="st" deviceset="STM32F103CX" device="TX"/>
 <part name="FRAME1" library="frames" deviceset="DINA3_L" device=""/>
 <part name="GND13" library="supply" deviceset="GND" device=""/>
@@
 <part name="P+2" library="supply" deviceset="+V" device=""/>
 <part name="GND20" library="supply" deviceset="GND" device=""/>
-<part name="U$7" library="freescale" deviceset="MC33962" device=""/>
 <part name="C13" library="rcl" deviceset="C-EU" device="C0603" value="100n"/>
 <part name="GND21" library="supply1" deviceset="GND" device=""/>
@@
 <part name="X4" library="con-molex" deviceset="53?-06" device="047"/>
 <part name="GND14" library="supply" deviceset="GND" device=""/>
+<part name="U$7" library="freescale" deviceset="MC33962" device=""/>
 </parts>
 <sheets>
@@
 <instance part="P+2" gate="1" x="312.42" y="152.4"/>
 <instance part="GND20" gate="1" x="312.42" y="137.16"/>
-<instance part="U$7" gate="G$1" x="223.52" y="185.42"/>
 <instance part="C13" gate="G$1" x="284.48" y="144.78"/>
 <instance part="GND21" gate="1" x="284.48" y="137.16"/>
@@
 <instance part="X4" gate="-6" x="233.68" y="96.52"/>
 <instance part="GND14" gate="1" x="294.64" y="137.16"/>
+<instance part="U$7" gate="G$1" x="223.52" y="185.42"/>
 </instances>
 <busses>
@@
 </segment>
 <segment>
-<pinref part="U$7" gate="G$1" pin="AGND"/>
 <pinref part="GND15" gate="1" pin="GND"/>
 <wire x1="241.3" y1="177.8" x2="243.84" y2="177.8" width="0.1524" layer="91"/>
 <wire x1="243.84" y1="177.8" x2="243.84" y2="175.26" width="0.1524" layer="91"/>
-<pinref part="U$7" gate="G$1" pin="PGND"/>
 <wire x1="243.84" y1="175.26" x2="243.84" y2="172.72" width="0.1524" layer="91"/>
 <wire x1="241.3" y1="175.26" x2="243.84" y2="175.26" width="0.1524" layer="91"/>
 <junction x="243.84" y="175.26"/>
+<pinref part="U$7" gate="G$1" pin="PGND"/>
+<pinref part="U$7" gate="G$1" pin="AGND"/>
 </segment>
 <segment>
@@
 <segment>
 <wire x1="241.3" y1="185.42" x2="243.84" y2="185.42" width="0.1524" layer="91"/>
+<label x="243.84" y="185.42" size="1.778" layer="95"/>
 <pinref part="U$7" gate="G$1" pin="OUT1"/>
-<label x="243.84" y="185.42" size="1.778" layer="95"/>
-</segment>
-<segment>
-<pinref part="X2" gate="-1" pin="S"/>
+</segment>
+<segment>
 <wire x1="314.96" y1="127" x2="309.88" y2="127" width="0.1524" layer="91"/>
 <label x="309.88" y="127" size="1.778" layer="95" rot="MR0"/>
+<pinref part="X2" gate="-1" pin="S"/>
 </segment>
 </net>
@@
 <segment>
 <wire x1="241.3" y1="182.88" x2="243.84" y2="182.88" width="0.1524" layer="91"/>
+<label x="243.84" y="182.88" size="1.778" layer="95"/>
 <pinref part="U$7" gate="G$1" pin="OUT2"/>
-<label x="243.84" y="182.88" size="1.778" layer="95"/>
-</segment>
-<segment>
-<pinref part="X2" gate="-2" pin="S"/>
+</segment>
+<segment>
 <wire x1="314.96" y1="124.46" x2="309.88" y2="124.46" width="0.1524" layer="91"/>
 <label x="309.88" y="124.46" size="1.778" layer="95" rot="MR0"/>
-</segment>
-</net>
-<net name="N$3" class="0">
-<segment>
-<pinref part="U$7" gate="G$1" pin="FB"/>
+<pinref part="X2" gate="-2" pin="S"/>
+</segment>
+</net>
+<net name="FB" class="0">
+<segment>
 <wire x1="205.74" y1="175.26" x2="200.66" y2="175.26" width="0.1524" layer="91"/>
 <pinref part="C15" gate="G$1" pin="1"/>
@@
 <junction x="193.04" y="175.26"/>
 <label x="187.96" y="175.26" size="1.778" layer="95" rot="MR0"/>
-</segment>
-</net>
-<net name="N$5" class="0">
-<segment>
+<pinref part="U$7" gate="G$1" pin="FB"/>
+</segment>
+</net>
+<net name="!SF" class="0">
+<segment>
+<wire x1="205.74" y1="177.8" x2="203.2" y2="177.8" width="0.1524" layer="91"/>
+<label x="203.2" y="177.8" size="1.778" layer="95" rot="MR0"/>
 <pinref part="U$7" gate="G$1" pin="!SF"/>
-<wire x1="205.74" y1="177.8" x2="203.2" y2="177.8" width="0.1524" layer="91"/>
-</segment>
-</net>
-<net name="N$9" class="0">
-<segment>
+</segment>
+</net>
+<net name="SLEW" class="0">
+<segment>
+<wire x1="205.74" y1="180.34" x2="203.2" y2="180.34" width="0.1524" layer="91"/>
+<label x="203.2" y="180.34" size="1.778" layer="95" rot="MR0"/>
 <pinref part="U$7" gate="G$1" pin="SLEW"/>
-<wire x1="205.74" y1="180.34" x2="203.2" y2="180.34" width="0.1524" layer="91"/>
-</segment>
-</net>
-<net name="N$10" class="0">
-<segment>
+</segment>
+</net>
+<net name="INV" class="0">
+<segment>
+<wire x1="205.74" y1="182.88" x2="203.2" y2="182.88" width="0.1524" layer="91"/>
+<label x="203.2" y="182.88" size="1.778" layer="95" rot="MR0"/>
 <pinref part="U$7" gate="G$1" pin="INV"/>
-<wire x1="205.74" y1="182.88" x2="203.2" y2="182.88" width="0.1524" layer="91"/>
-</segment>
-</net>
-<net name="N$11" class="0">
-<segment>
+</segment>
+</net>
+<net name="D1" class="0">
+<segment>
+<wire x1="205.74" y1="185.42" x2="203.2" y2="185.42" width="0.1524" layer="91"/>
+<label x="203.2" y="185.42" size="1.778" layer="95" rot="MR0"/>
 <pinref part="U$7" gate="G$1" pin="D1"/>
-<wire x1="205.74" y1="185.42" x2="203.2" y2="185.42" width="0.1524" layer="91"/>
-</segment>
-</net>
-<net name="N$12" class="0">
-<segment>
+</segment>
+</net>
+<net name="!D2" class="0">
+<segment>
+<wire x1="205.74" y1="187.96" x2="203.2" y2="187.96" width="0.1524" layer="91"/>
+<label x="203.2" y="187.96" size="1.778" layer="95" rot="MR0"/>
 <pinref part="U$7" gate="G$1" pin="!D2"/>
-<wire x1="205.74" y1="187.96" x2="203.2" y2="187.96" width="0.1524" layer="91"/>
-</segment>
-</net>
-<net name="N$13" class="0">
-<segment>
+</segment>
+</net>
+<net name="IN2" class="0">
+<segment>
+<wire x1="205.74" y1="190.5" x2="203.2" y2="190.5" width="0.1524" layer="91"/>
+<label x="203.2" y="190.5" size="1.778" layer="95" rot="MR0"/>
 <pinref part="U$7" gate="G$1" pin="IN2"/>
-<wire x1="205.74" y1="190.5" x2="203.2" y2="190.5" width="0.1524" layer="91"/>
-</segment>
-</net>
-<net name="N$14" class="0">
-<segment>
+</segment>
+</net>
+<net name="IN1" class="0">
+<segment>
+<wire x1="205.74" y1="193.04" x2="203.2" y2="193.04" width="0.1524" layer="91"/>
+<label x="203.2" y="193.04" size="1.778" layer="95" rot="MR0"/>
 <pinref part="U$7" gate="G$1" pin="IN1"/>
-<wire x1="205.74" y1="193.04" x2="203.2" y2="193.04" width="0.1524" layer="91"/>
-</segment>
-</net>
-<net name="N$15" class="0">
-<segment>
+</segment>
+</net>
+<net name="EN" class="0">
+<segment>
+<wire x1="205.74" y1="195.58" x2="203.2" y2="195.58" width="0.1524" layer="91"/>
+<label x="203.2" y="195.58" size="1.778" layer="95" rot="MR0"/>
 <pinref part="U$7" gate="G$1" pin="EN"/>
-<wire x1="205.74" y1="195.58" x2="203.2" y2="195.58" width="0.1524" layer="91"/>
-</segment>
-</net>
+</segment>
+</net>
