File: hw/uDC_module.sch (EAGLE design)
At the start: 38 parts, among them J1 GROVE-4P-2.0-3470130P1, J2 GROVE-4P-2.0-3470130P1, U5 LD3985XX, X1 22-23-2021, X2 22-23-2021, X3 53047-06, X4 53047-06

Commit message: small fixes for production
Parts:
- removed R3: 10k, rcl:R-EU_R0603
- added RN1: 4k7, dp_devices:RESISTOR_ARRAY_4
- added SJ1: SOLDERJUMPERTRACE, SparkFun:SOLDERJUMPERTRACE
Connections:
- removed net BOOT0: R3.2, U$6.BOOT0
- new net N$5: RN1A.2, RN1B.2, RN1C.2, SJ1.1
- net +3V3: now also SJ1.2
- net ENC_A: now also RN1B.1
- net ENC_B: now also RN1A.1
- net ENC_I: now also RN1C.1
- net GND: now also U$6.BOOT0; no longer R3.1
- net LED1: now also U$6.PD1/OSC_OUT; no longer U$6.PC13
Changed lines of the file:
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@@
 <?xml version="1.0" encoding="utf-8"?>
 <!DOCTYPE eagle SYSTEM "eagle.dtd">
-<eagle version="6.6.0">
+<eagle version="7.2.0">
 <drawing>
 <settings>
@@
 <part name="GND34" library="supply1" deviceset="GND" device=""/>
 <part name="+3V5" library="supply1" deviceset="+3V3" device=""/>
-<part name="R3" library="rcl" deviceset="R-EU_" device="R0603" value="10k"/>
 <part name="GND7" library="supply1" deviceset="GND" device=""/>
 <part name="+3V6" library="supply1" deviceset="+3V3" device=""/>
@@
 <part name="P+4" library="supply" deviceset="+5V" device=""/>
 <part name="GND33" library="supply1" deviceset="GND" device=""/>
+<part name="RN1" library="dp_devices" deviceset="RESISTOR_ARRAY_4" device="" value="4k7"/>
+<part name="+3V7" library="supply1" deviceset="+3V3" device=""/>
+<part name="SJ1" library="SparkFun" deviceset="SOLDERJUMPER" device="TRACE" value="SOLDERJUMPERTRACE"/>
 </parts>
 <sheets>
@@
 <instance part="GND34" gate="1" x="129.54" y="231.14"/>
 <instance part="+3V5" gate="G$1" x="93.98" y="180.34"/>
-<instance part="R3" gate="G$1" x="129.54" y="208.28" rot="R90"/>
-<instance part="GND7" gate="1" x="129.54" y="198.12"/>
+<instance part="GND7" gate="1" x="45.72" y="248.92" rot="R180"/>
 <instance part="+3V6" gate="G$1" x="134.62" y="165.1" rot="R270"/>
 <instance part="C3" gate="G$1" x="99.06" y="238.76"/>
@@
 <instance part="P+4" gate="1" x="228.6" y="116.84"/>
 <instance part="GND33" gate="1" x="276.86" y="91.44"/>
+<instance part="RN1" gate="B" x="220.98" y="111.76" rot="R90"/>
+<instance part="RN1" gate="C" x="210.82" y="111.76" rot="R90"/>
+<instance part="RN1" gate="D" x="175.26" y="83.82"/>
+<instance part="RN1" gate="A" x="215.9" y="111.76" rot="R90"/>
+<instance part="+3V7" gate="G$1" x="215.9" y="134.62"/>
+<instance part="SJ1" gate="1" x="215.9" y="124.46" rot="R90"/>
 </instances>
 <busses>
@@
 </segment>
 <segment>
-<pinref part="R3" gate="G$1" pin="1"/>
-<pinref part="GND7" gate="1" pin="GND"/>
-<wire x1="129.54" y1="200.66" x2="129.54" y2="203.2" width="0.1524" layer="91"/>
-</segment>
-<segment>
 <pinref part="C3" gate="G$1" pin="2"/>
 <pinref part="GND9" gate="1" pin="GND"/>
@@
 <wire x1="279.4" y1="96.52" x2="276.86" y2="96.52" width="0.1524" layer="91"/>
 <junction x="276.86" y="96.52"/>
+</segment>
+<segment>
+<pinref part="U$6" gate="G$1" pin="BOOT0"/>
+<pinref part="GND7" gate="1" pin="GND"/>
+<wire x1="45.72" y1="246.38" x2="45.72" y2="236.22" width="0.1524" layer="91"/>
 </segment>
 </net>
@@
 <pinref part="C18" gate="G$1" pin="1"/>
 </segment>
+<segment>
+<pinref part="SJ1" gate="1" pin="2"/>
+<pinref part="+3V7" gate="G$1" pin="+3V3"/>
+<wire x1="215.9" y1="132.08" x2="215.9" y2="129.54" width="0.1524" layer="91"/>
+</segment>
 </net>
 <net name="JTMS" class="0">
@@
 </segment>
 <segment>
-<pinref part="U$6" gate="G$1" pin="PC13"/>
-<wire x1="58.42" y1="236.22" x2="58.42" y2="238.76" width="0.1524" layer="91"/>
-<label x="58.42" y="238.76" size="1.778" layer="95" rot="R90"/>
+<wire x1="48.26" y1="236.22" x2="48.26" y2="238.76" width="0.1524" layer="91"/>
+<label x="48.26" y="238.76" size="1.778" layer="95" rot="R90"/>
+<pinref part="U$6" gate="G$1" pin="PD1/OSC_OUT"/>
 </segment>
 </net>
@@
 <label x="86.36" y="215.9" size="1.778" layer="95"/>
 <pinref part="U$6" gate="G$1" pin="PB9"/>
-</segment>
-</net>
-<net name="BOOT0" class="0">
-<segment>
-<wire x1="45.72" y1="236.22" x2="45.72" y2="238.76" width="0.1524" layer="91"/>
-<label x="45.72" y="238.76" size="1.778" layer="95" rot="R90"/>
-<pinref part="U$6" gate="G$1" pin="BOOT0"/>
-</segment>
-<segment>
-<wire x1="121.92" y1="215.9" x2="129.54" y2="215.9" width="0.1524" layer="91"/>
-<wire x1="129.54" y1="215.9" x2="129.54" y2="213.36" width="0.1524" layer="91"/>
-<pinref part="R3" gate="G$1" pin="2"/>
-<label x="114.3" y="215.9" size="1.778" layer="95"/>
 </segment>
 </net>
@@
 <segment>
 <pinref part="X4" gate="-3" pin="S"/>
-<wire x1="231.14" y1="104.14" x2="226.06" y2="104.14" width="0.1524" layer="91"/>
-<label x="226.06" y="104.14" size="1.778" layer="95" rot="MR0"/>
+<wire x1="231.14" y1="104.14" x2="220.98" y2="104.14" width="0.1524" layer="91"/>
+<label x="205.74" y="104.14" size="1.778" layer="95" rot="MR0"/>
+<pinref part="RN1" gate="B" pin="1"/>
+<wire x1="220.98" y1="104.14" x2="205.74" y2="104.14" width="0.1524" layer="91"/>
+<wire x1="220.98" y1="106.68" x2="220.98" y2="104.14" width="0.1524" layer="91"/>
+<junction x="220.98" y="104.14"/>
 </segment>
 <segment>
@@
 <segment>
 <pinref part="X4" gate="-4" pin="S"/>
-<wire x1="231.14" y1="101.6" x2="226.06" y2="101.6" width="0.1524" layer="91"/>
-<label x="226.06" y="101.6" size="1.778" layer="95" rot="MR0"/>
+<wire x1="231.14" y1="101.6" x2="215.9" y2="101.6" width="0.1524" layer="91"/>
+<label x="205.74" y="101.6" size="1.778" layer="95" rot="MR0"/>
+<pinref part="RN1" gate="A" pin="1"/>
+<wire x1="215.9" y1="101.6" x2="205.74" y2="101.6" width="0.1524" layer="91"/>
+<wire x1="215.9" y1="106.68" x2="215.9" y2="101.6" width="0.1524" layer="91"/>
+<junction x="215.9" y="101.6"/>
 </segment>
 <segment>
@@
 <segment>
 <pinref part="X4" gate="-5" pin="S"/>
-<wire x1="231.14" y1="99.06" x2="226.06" y2="99.06" width="0.1524" layer="91"/>
-<label x="226.06" y="99.06" size="1.778" layer="95" rot="MR0"/>
+<wire x1="231.14" y1="99.06" x2="210.82" y2="99.06" width="0.1524" layer="91"/>
+<label x="205.74" y="99.06" size="1.778" layer="95" rot="MR0"/>
+<pinref part="RN1" gate="C" pin="1"/>
+<wire x1="210.82" y1="99.06" x2="205.74" y2="99.06" width="0.1524" layer="91"/>
+<wire x1="210.82" y1="106.68" x2="210.82" y2="99.06" width="0.1524" layer="91"/>
+<junction x="210.82" y="99.06"/>
 </segment>
 <segment>
@@
 </segment>
 </net>
+<net name="N$5" class="0">
+<segment>
+<pinref part="RN1" gate="B" pin="2"/>
+<wire x1="220.98" y1="116.84" x2="220.98" y2="119.38" width="0.1524" layer="91"/>
+<wire x1="220.98" y1="119.38" x2="215.9" y2="119.38" width="0.1524" layer="91"/>
+<pinref part="RN1" gate="C" pin="2"/>
+<wire x1="210.82" y1="116.84" x2="210.82" y2="119.38" width="0.1524" layer="91"/>
+<wire x1="210.82" y1="119.38" x2="215.9" y2="119.38" width="0.1524" layer="91"/>
+<junction x="215.9" y="119.38"/>
+<pinref part="RN1" gate="A" pin="2"/>
+<wire x1="215.9" y1="116.84" x2="215.9" y2="119.38" width="0.1524" layer="91"/>
+<pinref part="SJ1" gate="1" pin="1"/>
+</segment>
+</net>
